Commit message: Adding Submodel

File: src/project_pkg/urdf/project_pkg.urdf (robot description, URDF)
Before this commit: robot project_pkg, 6 links, 5 joints
Links:
- added link map
- added link odom
Joints:
- added joint map_joint: type fixed, parent base_link, child map, origin xyz=0 0 0 rpy=0 0 0
- added joint odom_joint: type fixed, parent base_link, child odom, origin xyz=0 0 0 rpy=0 0 0
